File: CESP.sch (KiCad schematic (older format))
At the start: 5 parts

Commit message: Laid out a PCB with all required component types.
Parts:
- removed U?: LTC1594CS, TSSOP14, symbol LTC1594CS
- removed U?: TL074, TSSOP14, symbol TL074
- removed U? (x3): TL074, symbol TL074
- added C1, C2, C3: C, ~, symbol C
- added D1: DIODE, ~, symbol DIODE
- added D2: LED, ~, symbol LED
- added D3: ZENER, ~, symbol ZENER
- added Q1, Q2: PN2222A, TO92, symbol PN2222A
- added Q3: MOSFET_N, ~, symbol MOSFET_N
- added R1, R2, R3, R4: R, ~, symbol R
- added SW1: SW_PUSH, ~, symbol SW_PUSH
- added U1: LM324, symbol LM324
Connections:
- net labels added: +12V, -12V, GND, VCC
- wire segments 0 -> 35
Other:
- note removed: "NOTE: THIS IS JUST A TEST BOARD\nREMOVE ALL COMPONENTS AND CREATE YOUR OWN\nINCLUDE SCHEMATIC HOOKUPS/NETLIST"
